File: hardware/terminal/terminal.sch (KiCad schematic (older format))
At the start: 12 parts

Commit message: o Add programming header.
Parts:
- added P?: Prog, symbol CONN_5
- added R?: 2.2k, symbol R
Connections:
- net labels added: MISO, MOSI, SCK
- wire segments 45 -> 40

Commit message: o Initial annotations.
Parts:
- gave numbers to parts that had none: 14
Connections:
- wire segments 40 -> 41
Other:
- note added: "RX"
- note added: "TX"
Changed lines of the file:
@@
 $EndDescr
 $Comp
-L MAX232 U?
+L MAX232 U2
 U 1 1 53EB8217
 P 7900 2700
-F 0 "U?" H 7900 3550 70  0000 C CNN
+F 0 "U2" H 7900 3550 70  0000 C CNN
 F 1 "MAX232" H 7900 1850 70  0000 C CNN
 F 2 "" H 7900 2700 60  0000 C CNN
@@
 $EndComp
 $Comp
-L C C?
+L C C1
 U 1 1 53EB8368
 P 7000 2200
-F 0 "C?" H 7050 2300 50  0000 L CNN
+F 0 "C1" H 7050 2300 50  0000 L CNN
 F 1 "C" H 7050 2100 50  0000 L CNN
 F 2 "" H 7000 2200 60  0000 C CNN
@@
 $EndComp
 $Comp
-L C C?
+L C C2
 U 1 1 53EB837C
 P 7000 2700
-F 0 "C?" H 7050 2800 50  0000 L CNN
+F 0 "C2" H 7050 2800 50  0000 L CNN
 F 1 "C" H 7050 2600 50  0000 L CNN
 F 2 "" H 7000 2700 60  0000 C CNN
@@
 $EndComp
 $Comp
-L C C?
+L C C3
 U 1 1 53EB8390
 P 8900 2400
-F 0 "C?" H 8950 2500 50  0000 L CNN
+F 0 "C3" H 8950 2500 50  0000 L CNN
 F 1 "C" H 8950 2300 50  0000 L CNN
 F 2 "" H 8900 2400 60  0000 C CNN
@@
 $EndComp
 $Comp
-L C C?
+L C C4
 U 1 1 53EB83A4
 P 8900 2900
-F 0 "C?" H 8950 3000 50  0000 L CNN
+F 0 "C4" H 8950 3000 50  0000 L CNN
 F 1 "C" H 8950 2800 50  0000 L CNN
 F 2 "" H 8900 2900 60  0000 C CNN
@@
 $EndComp
 $Comp
-L GND #PWR?
+L GND #PWR20
 U 1 1 53EB83C0
 P 9250 2700
-F 0 "#PWR?" H 9250 2700 30  0001 C CNN
+F 0 "#PWR20" H 9250 2700 30  0001 C CNN
 F 1 "GND" H 9250 2630 30  0001 C CNN
 F 2 "" H 9250 2700 60  0000 C CNN
@@
 	7000 2900 7100 2900
 $Comp
-L +3.3V #PWR?
+L +3.3V #PWR16
 U 1 1 53EB841D
 P 8750 2000
-F 0 "#PWR?" H 8750 1960 30  0001 C CNN
+F 0 "#PWR16" H 8750 1960 30  0001 C CNN
 F 1 "+3.3V" H 8750 2110 30  0000 C CNN
 F 2 "" H 8750 2000 60  0000 C CNN
@@
 RX
 $Comp
-L ATMEGA8-P IC?
+L ATMEGA8-P IC1
 U 1 1 53EB84A5
 P 3050 3200
-F 0 "IC?" H 2350 4450 50  0000 L BNN
+F 0 "IC1" H 2350 4450 50  0000 L BNN
 F 1 "ATMEGA8-P" H 3400 1800 50  0000 L BNN
 F 2 "DIL28" H 2450 1850 50  0001 C CNN
@@
 $EndComp
 $Comp
-L RJ45 J?
+L RJ45 J1
 U 1 1 53EB84C6
 P 9800 3450
-F 0 "J?" H 10000 3950 60  0000 C CNN
+F 0 "J1" H 10000 3950 60  0000 C CNN
 F 1 "RJ45" H 9650 3950 60  0000 C CNN
 F 2 "" H 9800 3450 60  0000 C CNN
@@
 TX
 $Comp
-L +12V #PWR?
+L +12V #PWR17
 U 1 1 53EB8601
 P 8800 3700
-F 0 "#PWR?" H 8800 3650 20  0001 C CNN
+F 0 "#PWR17" H 8800 3650 20  0001 C CNN
 F 1 "+12V" H 8800 3800 30  0000 C CNN
 F 2 "" H 8800 3700 60  0000 C CNN
@@
 	9200 3500 9350 3500
 $Comp
-L CONN_8 P?
+L CONN_8 P2
 U 1 1 53EB87E0
 P 5600 2400
-F 0 "P?" V 5550 2400 60  0000 C CNN
+F 0 "P2" V 5550 2400 60  0000 C CNN
 F 1 "RC522" V 5650 2400 60  0000 C CNN
 F 2 "" H 5600 2400 60  0000 C CNN
@@
 $EndComp
 $Comp
-L 7805 U?
+L 7805 U3
 U 1 1 53EB87F5
 P 9000 4200
-F 0 "U?" H 9150 4004 60  0000 C CNN
+F 0 "U3" H 9150 4004 60  0000 C CNN
 F 1 "7803" H 9000 4400 60  0000 C CNN
 F 2 "" H 9000 4200 60  0000 C CNN
@@
 $EndComp
 $Comp
-L GND #PWR?
+L GND #PWR22
 U 1 1 53EB881B
 P 10150 4000
-F 0 "#PWR?" H 10150 4000 30  0001 C CNN
+F 0 "#PWR22" H 10150 4000 30  0001 C CNN
 F 1 "GND" H 10150 3930 30  0001 C CNN
 F 2 "" H 10150 4000 60  0000 C CNN
@@
 $EndComp
 $Comp
-L +12V #PWR?
+L +12V #PWR15
 U 1 1 53EB882F
 P 8600 4100
-F 0 "#PWR?" H 8600 4050 20  0001 C CNN
+F 0 "#PWR15" H 8600 4050 20  0001 C CNN
 F 1 "+12V" H 8600 4200 30  0000 C CNN
 F 2 "" H 8600 4100 60  0000 C CNN
@@
 	8600 4100 8600 4150
 $Comp
-L GND #PWR?
+L GND #PWR18
 U 1 1 53EB884F
 P 9000 4450
-F 0 "#PWR?" H 9000 4450 30  0001 C CNN
+F 0 "#PWR18" H 9000 4450 30  0001 C CNN
 F 1 "GND" H 9000 4380 30  0001 C CNN
 F 2 "" H 9000 4450 60  0000 C CNN
@@
 $EndComp
 $Comp
-L +3.3V #PWR?
+L +3.3V #PWR21
 U 1 1 53EB8966
 P 9400 4100
-F 0 "#PWR?" H 9400 4060 30  0001 C CNN
+F 0 "#PWR21" H 9400 4060 30  0001 C CNN
 F 1 "+3.3V" H 9400 4210 30  0000 C CNN
 F 2 "" H 9400 4100 60  0000 C CNN
@@
 	9400 4150 9400 4100
 $Comp
-L +3.3V #PWR?
+L +3.3V #PWR8
 U 1 1 53EB89B2
 P 5250 2000
-F 0 "#PWR?" H 5250 1960 30  0001 C CNN
+F 0 "#PWR8" H 5250 1960 30  0001 C CNN
 F 1 "+3.3V" H 5250 2110 30  0000 C CNN
 F 2 "" H 5250 2000 60  0000 C CNN
@@
 	4050 2200 4450 2200
 $Comp
-L GND #PWR?
+L GND #PWR4
 U 1 1 53EB89F8
 P 5100 2300
-F 0 "#PWR?" H 5100 2300 30  0001 C CNN
+F 0 "#PWR4" H 5100 2300 30  0001 C CNN
 F 1 "GND" H 5100 2230 30  0001 C CNN
 F 2 "" H 5100 2300 60  0000 C CNN
@@
 $EndComp
 $Comp
-L GND #PWR?
+L GND #PWR2
 U 1 1 53EB8B64
 P 3050 4700
-F 0 "#PWR?" H 3050 4700 30  0001 C CNN
+F 0 "#PWR2" H 3050 4700 30  0001 C CNN
 F 1 "GND" H 3050 4630 30  0001 C CNN
 F 2 "" H 3050 4700 60  0000 C CNN
@@
 $EndComp
 $Comp
-L +3.3V #PWR?
+L +3.3V #PWR1
 U 1 1 53EB8B76
 P 3050 1800
-F 0 "#PWR?" H 3050 1760 30  0001 C CNN
+F 0 "#PWR1" H 3050 1760 30  0001 C CNN
 F 1 "+3.3V" H 3050 1910 30  0000 C CNN
 F 2 "" H 3050 1800 60  0000 C CNN
@@
 $EndComp
 $Comp
-L CONN_8X2 P?
+L CONN_8X2 P3
 U 1 1 53EB8E37
 P 5600 3400
-F 0 "P?" H 5600 3850 60  0000 C CNN
+F 0 "P3" H 5600 3850 60  0000 C CNN
 F 1 "LCD" V 5600 3400 50  0000 C CNN
 F 2 "" H 5600 3400 60  0000 C CNN
@@
 $EndComp
 $Comp
-L CONN_8X2 P?
+L CONN_8X2 P4
 U 1 1 53EB8E91
 P 5600 4350
-F 0 "P?" H 5600 4800 60  0000 C CNN
+F 0 "P4" H 5600 4800 60  0000 C CNN
 F 1 "Keypad" V 5600 4350 50  0000 C CNN
 F 2 "" H 5600 4350 60  0000 C CNN
@@
 $EndComp
 $Comp
-L 7805 U?
+L 7805 U1
 U 1 1 53EC1B60
 P 7750 4200
-F 0 "U?" H 7900 4004 60  0000 C CNN
+F 0 "U1" H 7900 4004 60  0000 C CNN
 F 1 "7805" H 7750 4400 60  0000 C CNN
 F 2 "" H 7750 4200 60  0000 C CNN
@@
 $EndComp
 $Comp
-L +12V #PWR?
+L +12V #PWR12
 U 1 1 53EC1B72
 P 7350 4100
-F 0 "#PWR?" H 7350 4050 20  0001 C CNN
+F 0 "#PWR12" H 7350 4050 20  0001 C CNN
 F 1 "+12V" H 7350 4200 30  0000 C CNN
 F 2 "" H 7350 4100 60  0000 C CNN
@@
 	7350 4100 7350 4150
 $Comp
-L +5V #PWR?
+L +5V #PWR14
 U 1 1 53EC1BA0
 P 8150 4100
-F 0 "#PWR?" H 8150 4190 20  0001 C CNN
+F 0 "#PWR14" H 8150 4190 20  0001 C CNN
 F 1 "+5V" H 8150 4190 30  0000 C CNN
 F 2 "" H 8150 4100 60  0000 C CNN
@@
 	8150 4100 8150 4150
 $Comp
-L GND #PWR?
+L GND #PWR13
 U 1 1 53EC1BD4
 P 7750 4450
-F 0 "#PWR?" H 7750 4450 30  0001 C CNN
+F 0 "#PWR13" H 7750 4450 30  0001 C CNN
 F 1 "GND" H 7750 4380 30  0001 C CNN
 F 2 "" H 7750 4450 60  0000 C CNN
@@
 $EndComp
 $Comp
-L GND #PWR?
+L GND #PWR5
 U 1 1 53EC1BE1
 P 5200 3050
-F 0 "#PWR?" H 5200 3050 30  0001 C CNN
+F 0 "#PWR5" H 5200 3050 30  0001 C CNN
 F 1 "GND" H 5200 2980 30  0001 C CNN
 F 2 "" H 5200 3050 60  0000 C CNN
@@
 $EndComp
 $Comp
-L +5V #PWR?
+L +5V #PWR9
 U 1 1 53EC1BF5
 P 6000 3050
-F 0 "#PWR?" H 6000 3140 20  0001 C CNN
+F 0 "#PWR9" H 6000 3140 20  0001 C CNN
 F 1 "+5V" H 6000 3140 30  0000 C CNN
 F 2 "" H 6000 3050 60  0000 C CNN
@@
 $EndComp
 $Comp
-L GND #PWR?
+L GND #PWR6
 U 1 1 53EC1C07
 P 5200 3150
-F 0 "#PWR?" H 5200 3150 30  0001 C CNN
+F 0 "#PWR6" H 5200 3150 30  0001 C CNN
 F 1 "GND" H 5200 3080 30  0001 C CNN
 F 2 "" H 5200 3150 60  0000 C CNN
@@
 LCD-RS
 $Comp
-L GND #PWR?
+L GND #PWR7
 U 1 1 53EC1C74
 P 5200 3250
-F 0 "#PWR?" H 5200 3250 30  0001 C CNN
+F 0 "#PWR7" H 5200 3250 30  0001 C CNN
 F 1 "GND" H 5200 3180 30  0001 C CNN
 F 2 "" H 5200 3250 60  0000 C CNN
@@
 LCD-D3
 $Comp
-L GND #PWR?
+L GND #PWR10
 U 1 1 53EC1E47
 P 6000 4800
-F 0 "#PWR?" H 6000 4800 30  0001 C CNN
+F 0 "#PWR10" H 6000 4800 30  0001 C CNN
 F 1 "GND" H 6000 4730 30  0001 C CNN
 F 2 "" H 6000 4800 60  0000 C CNN
@@
 	4450 2150 5250 2150
 $Comp
-L GND #PWR?
+L GND #PWR11
 U 1 1 53EC2288
 P 6850 3500
-F 0 "#PWR?" H 6850 3500 30  0001 C CNN
+F 0 "#PWR11" H 6850 3500 30  0001 C CNN
 F 1 "GND" H 6850 3430 30  0001 C CNN
 F 2 "" H 6850 3500 60  0000 C CNN
@@
 	9350 3400 9200 3400
 $Comp
-L GND #PWR?
+L GND #PWR19
 U 1 1 53EC2456
 P 9150 3450
-F 0 "#PWR?" H 9150 3450 30  0001 C CNN
+F 0 "#PWR19" H 9150 3450 30  0001 C CNN
 F 1 "GND" H 9150 3380 30  0001 C CNN
 F 2 "" H 9150 3450 60  0000 C CNN
@@
 	9150 3300 9350 3300
 $Comp
-L CONN_5 P?
+L CONN_5 P1
 U 1 1 53ECE73B
 P 5000 1550
-F 0 "P?" V 4950 1550 50  0000 C CNN
+F 0 "P1" V 4950 1550 50  0000 C CNN
 F 1 "Prog" V 5050 1550 50  0000 C CNN
 F 2 "" H 5000 1550 60  0000 C CNN
@@
 $EndComp
 $Comp
-L GND #PWR?
+L GND #PWR3
 U 1 1 53ECE752
 P 4600 1800
-F 0 "#PWR?" H 4600 1800 30  0001 C CNN
+F 0 "#PWR3" H 4600 1800 30  0001 C CNN
 F 1 "GND" H 4600 1730 30  0001 C CNN
 F 2 "" H 4600 1800 60  0000 C CNN
@@
 	2150 1350 4600 1350
 $Comp
-L R R?
+L R R1
 U 1 1 53ECE910
 P 4850 2500
-F 0 "R?" V 4930 2500 50  0000 C CNN
+F 0 "R1" V 4930 2500 50  0000 C CNN
 F 1 "2.2k" V 4850 2500 50  0000 C CNN
 F 2 "" H 4850 2500 60  0000 C CNN
@@
 Wire Wire Line
 	4850 2050 5250 2050
+Text Notes 9500 3300 0    60   ~ 0
+TX
+Text Notes 9500 3650 0    60   ~ 0
+RX
+$Comp
+L GND #PWR?
+U 1 1 53ED5509
+P 8700 3500
+F 0 "#PWR?" H 8700 3500 30  0001 C CNN
+F 1 "GND" H 8700 3430 30  0001 C CNN
+F 2 "" H 8700 3500 60  0000 C CNN
+F 3 "" H 8700 3500 60  0000 C CNN
+	1    8700 3500
+	1    0    0    -1
+$EndComp
+Wire Wire Line
+	8700 3400 8700 3500
 $EndSCHEMATC

Commit message: o Add initial board.
Parts:
- C1, C2, C3, C4: footprint (none) -> Capacitors_SMD:c_0805
- IC1: footprint DIL28 -> Sockets_DIP:DIP-28__300
- J1: footprint (none) -> Connect:RJ45_8
- P1: footprint (none) -> Connect:SIL-5
- P2: footprint (none) -> Connect:SIL-8
- P3, P4: footprint (none) -> Pin_Headers:Pin_Header_Straight_2x08
- R1: footprint (none) -> SMD_Packages:SMD-0805
- U1, U3: footprint (none) -> Discret:LM78XXV
- U2: footprint (none) -> SMD_Packages:TSSOP-16
Changed lines of the file:
@@
 EESchema Schematic File Version 2
+LIBS:74xx
+LIBS:adc-dac
+LIBS:analog_switches
+LIBS:atmel
+LIBS:audio
+LIBS:cmos4000
+LIBS:conn
+LIBS:contrib
+LIBS:cypress
+LIBS:device
+LIBS:digital-audio
+LIBS:display
+LIBS:dsp
+LIBS:intel
+LIBS:interface
+LIBS:linear
+LIBS:memory
+LIBS:microchip
+LIBS:microcontrollers
+LIBS:motorola
+LIBS:opto
+LIBS:philips
 LIBS:power
-LIBS:device
+LIBS:regul
+LIBS:siliconi
+LIBS:special
+LIBS:texas
 LIBS:transistors
-LIBS:conn
-LIBS:linear
-LIBS:regul
-LIBS:74xx
-LIBS:cmos4000
-LIBS:adc-dac
-LIBS:memory
+LIBS:valves
 LIBS:xilinx
-LIBS:special
-LIBS:microcontrollers
-LIBS:dsp
-LIBS:microchip
-LIBS:analog_switches
-LIBS:motorola
-LIBS:texas
-LIBS:intel
-LIBS:audio
-LIBS:interface
-LIBS:digital-audio
-LIBS:philips
-LIBS:display
-LIBS:cypress
-LIBS:siliconi
-LIBS:opto
-LIBS:atmel
-LIBS:contrib
-LIBS:valves
 LIBS:terminal-cache
 EELAYER 24 0
@@
 F 0 "U2" H 7900 3550 70  0000 C CNN
 F 1 "MAX232" H 7900 1850 70  0000 C CNN
-F 2 "" H 7900 2700 60  0000 C CNN
+F 2 "SMD_Packages:TSSOP-16" H 7900 2700 60  0000 C CNN
 F 3 "" H 7900 2700 60  0000 C CNN
 	1    7900 2700
@@
 F 0 "C1" H 7050 2300 50  0000 L CNN
 F 1 "C" H 7050 2100 50  0000 L CNN
-F 2 "" H 7000 2200 60  0000 C CNN
+F 2 "Capacitors_SMD:c_0805" H 7000 2200 60  0000 C CNN
 F 3 "" H 7000 2200 60  0000 C CNN
 	1    7000 2200
@@
 F 0 "C2" H 7050 2800 50  0000 L CNN
 F 1 "C" H 7050 2600 50  0000 L CNN
-F 2 "" H 7000 2700 60  0000 C CNN
+F 2 "Capacitors_SMD:c_0805" H 7000 2700 60  0000 C CNN
 F 3 "" H 7000 2700 60  0000 C CNN
 	1    7000 2700
@@
 F 0 "C3" H 8950 2500 50  0000 L CNN
 F 1 "C" H 8950 2300 50  0000 L CNN
-F 2 "" H 8900 2400 60  0000 C CNN
+F 2 "Capacitors_SMD:c_0805" H 8900 2400 60  0000 C CNN
 F 3 "" H 8900 2400 60  0000 C CNN
 	1    8900 2400
@@
 F 0 "C4" H 8950 3000 50  0000 L CNN
 F 1 "C" H 8950 2800 50  0000 L CNN
-F 2 "" H 8900 2900 60  0000 C CNN
+F 2 "Capacitors_SMD:c_0805" H 8900 2900 60  0000 C CNN
 F 3 "" H 8900 2900 60  0000 C CNN
 	1    8900 2900
@@
 $EndComp
 $Comp
-L GND #PWR20
+L GND #PWR01
 U 1 1 53EB83C0
 P 9250 2700
-F 0 "#PWR20" H 9250 2700 30  0001 C CNN
+F 0 "#PWR01" H 9250 2700 30  0001 C CNN
 F 1 "GND" H 9250 2630 30  0001 C CNN
 F 2 "" H 9250 2700 60  0000 C CNN
@@
 	7000 2900 7100 2900
 $Comp
-L +3.3V #PWR16
+L +3.3V #PWR02
 U 1 1 53EB841D
 P 8750 2000
-F 0 "#PWR16" H 8750 1960 30  0001 C CNN
+F 0 "#PWR02" H 8750 1960 30  0001 C CNN
 F 1 "+3.3V" H 8750 2110 30  0000 C CNN
 F 2 "" H 8750 2000 60  0000 C CNN
@@
 F 0 "IC1" H 2350 4450 50  0000 L BNN
 F 1 "ATMEGA8-P" H 3400 1800 50  0000 L BNN
-F 2 "DIL28" H 2450 1850 50  0001 C CNN
+F 2 "Sockets_DIP:DIP-28__300" H 2450 1850 50  0001 C CNN
 F 3 "" H 3050 3200 60  0000 C CNN
 	1    3050 3200
@@
 F 0 "J1" H 10000 3950 60  0000 C CNN
 F 1 "RJ45" H 9650 3950 60  0000 C CNN
-F 2 "" H 9800 3450 60  0000 C CNN
+F 2 "Connect:RJ45_8" H 9800 3450 60  0000 C CNN
 F 3 "" H 9800 3450 60  0000 C CNN
 	1    9800 3450
@@
 TX
 $Comp
-L +12V #PWR17
+L +12V #PWR03
 U 1 1 53EB8601
 P 8800 3700
-F 0 "#PWR17" H 8800 3650 20  0001 C CNN
+F 0 "#PWR03" H 8800 3650 20  0001 C CNN
 F 1 "+12V" H 8800 3800 30  0000 C CNN
 F 2 "" H 8800 3700 60  0000 C CNN
@@
 F 0 "P2" V 5550 2400 60  0000 C CNN
 F 1 "RC522" V 5650 2400 60  0000 C CNN
-F 2 "" H 5600 2400 60  0000 C CNN
+F 2 "Connect:SIL-8" H 5600 2400 60  0000 C CNN
 F 3 "" H 5600 2400 60  0000 C CNN
 	1    5600 2400
@@
 F 0 "U3" H 9150 4004 60  0000 C CNN
 F 1 "7803" H 9000 4400 60  0000 C CNN
-F 2 "" H 9000 4200 60  0000 C CNN
+F 2 "Discret:LM78XXV" H 9000 4200 60  0000 C CNN
 F 3 "" H 9000 4200 60  0000 C CNN
 	1    9000 4200
@@
 $EndComp
 $Comp
-L GND #PWR22
+L GND #PWR04
 U 1 1 53EB881B
 P 10150 4000
-F 0 "#PWR22" H 10150 4000 30  0001 C CNN
+F 0 "#PWR04" H 10150 4000 30  0001 C CNN
 F 1 "GND" H 10150 3930 30  0001 C CNN
 F 2 "" H 10150 4000 60  0000 C CNN
@@
 $EndComp
 $Comp
-L +12V #PWR15
+L +12V #PWR05
 U 1 1 53EB882F
 P 8600 4100
-F 0 "#PWR15" H 8600 4050 20  0001 C CNN
+F 0 "#PWR05" H 8600 4050 20  0001 C CNN
 F 1 "+12V" H 8600 4200 30  0000 C CNN
 F 2 "" H 8600 4100 60  0000 C CNN
@@
 	8600 4100 8600 4150
 $Comp
-L GND #PWR18
+L GND #PWR06
 U 1 1 53EB884F
 P 9000 4450
-F 0 "#PWR18" H 9000 4450 30  0001 C CNN
+F 0 "#PWR06" H 9000 4450 30  0001 C CNN
 F 1 "GND" H 9000 4380 30  0001 C CNN
 F 2 "" H 9000 4450 60  0000 C CNN
@@
 $EndComp
 $Comp
-L +3.3V #PWR21
+L +3.3V #PWR07
 U 1 1 53EB8966
 P 9400 4100
-F 0 "#PWR21" H 9400 4060 30  0001 C CNN
+F 0 "#PWR07" H 9400 4060 30  0001 C CNN
 F 1 "+3.3V" H 9400 4210 30  0000 C CNN
 F 2 "" H 9400 4100 60  0000 C CNN
@@
 	9400 4150 9400 4100
 $Comp
-L +3.3V #PWR8
+L +3.3V #PWR08
 U 1 1 53EB89B2
 P 5250 2000
-F 0 "#PWR8" H 5250 1960 30  0001 C CNN
+F 0 "#PWR08" H 5250 1960 30  0001 C CNN
 F 1 "+3.3V" H 5250 2110 30  0000 C CNN
 F 2 "" H 5250 2000 60  0000 C CNN
@@
 	4050 2200 4450 2200
 $Comp
-L GND #PWR4
+L GND #PWR09
 U 1 1 53EB89F8
 P 5100 2300
-F 0 "#PWR4" H 5100 2300 30  0001 C CNN
+F 0 "#PWR09" H 5100 2300 30  0001 C CNN
 F 1 "GND" H 5100 2230 30  0001 C CNN
 F 2 "" H 5100 2300 60  0000 C CNN
@@
 $EndComp
 $Comp
-L GND #PWR2
+L GND #PWR010
 U 1 1 53EB8B64
 P 3050 4700
-F 0 "#PWR2" H 3050 4700 30  0001 C CNN
+F 0 "#PWR010" H 3050 4700 30  0001 C CNN
 F 1 "GND" H 3050 4630 30  0001 C CNN
 F 2 "" H 3050 4700 60  0000 C CNN
@@
 $EndComp
 $Comp
-L +3.3V #PWR1
+L +3.3V #PWR011
 U 1 1 53EB8B76
 P 3050 1800
-F 0 "#PWR1" H 3050 1760 30  0001 C CNN
+F 0 "#PWR011" H 3050 1760 30  0001 C CNN
 F 1 "+3.3V" H 3050 1910 30  0000 C CNN
 F 2 "" H 3050 1800 60  0000 C CNN
@@
 F 0 "P3" H 5600 3850 60  0000 C CNN
 F 1 "LCD" V 5600 3400 50  0000 C CNN
-F 2 "" H 5600 3400 60  0000 C CNN
+F 2 "Pin_Headers:Pin_Header_Straight_2x08" H 5600 3400 60  0000 C CNN
 F 3 "" H 5600 3400 60  0000 C CNN
 	1    5600 3400
@@
 F 0 "P4" H 5600 4800 60  0000 C CNN
 F 1 "Keypad" V 5600 4350 50  0000 C CNN
-F 2 "" H 5600 4350 60  0000 C CNN
+F 2 "Pin_Headers:Pin_Header_Straight_2x08" H 5600 4350 60  0000 C CNN
 F 3 "" H 5600 4350 60  0000 C CNN
 	1    5600 4350
@@
 F 0 "U1" H 7900 4004 60  0000 C CNN
 F 1 "7805" H 7750 4400 60  0000 C CNN
-F 2 "" H 7750 4200 60  0000 C CNN
+F 2 "Discret:LM78XXV" H 7750 4200 60  0000 C CNN
 F 3 "" H 7750 4200 60  0000 C CNN
 	1    7750 4200
@@
 $EndComp
 $Comp
-L +12V #PWR12
+L +12V #PWR012
 U 1 1 53EC1B72
 P 7350 4100
-F 0 "#PWR12" H 7350 4050 20  0001 C CNN
+F 0 "#PWR012" H 7350 4050 20  0001 C CNN
 F 1 "+12V" H 7350 4200 30  0000 C CNN
 F 2 "" H 7350 4100 60  0000 C CNN
@@
 	7350 4100 7350 4150
 $Comp
-L +5V #PWR14
+L +5V #PWR013
 U 1 1 53EC1BA0
 P 8150 4100
-F 0 "#PWR14" H 8150 4190 20  0001 C CNN
+F 0 "#PWR013" H 8150 4190 20  0001 C CNN
 F 1 "+5V" H 8150 4190 30  0000 C CNN
 F 2 "" H 8150 4100 60  0000 C CNN
@@
 	8150 4100 8150 4150
 $Comp
-L GND #PWR13
+L GND #PWR014
 U 1 1 53EC1BD4
 P 7750 4450
-F 0 "#PWR13" H 7750 4450 30  0001 C CNN
+F 0 "#PWR014" H 7750 4450 30  0001 C CNN
 F 1 "GND" H 7750 4380 30  0001 C CNN
 F 2 "" H 7750 4450 60  0000 C CNN
@@
 $EndComp
 $Comp
-L GND #PWR5
+L GND #PWR015
 U 1 1 53EC1BE1
 P 5200 3050
-F 0 "#PWR5" H 5200 3050 30  0001 C CNN
+F 0 "#PWR015" H 5200 3050 30  0001 C CNN
 F 1 "GND" H 5200 2980 30  0001 C CNN
 F 2 "" H 5200 3050 60  0000 C CNN
@@
 $EndComp
 $Comp
-L +5V #PWR9
+L +5V #PWR016
 U 1 1 53EC1BF5
 P 6000 3050
-F 0 "#PWR9" H 6000 3140 20  0001 C CNN
+F 0 "#PWR016" H 6000 3140 20  0001 C CNN
 F 1 "+5V" H 6000 3140 30  0000 C CNN
 F 2 "" H 6000 3050 60  0000 C CNN
@@
 $EndComp
 $Comp
-L GND #PWR6
+L GND #PWR017
 U 1 1 53EC1C07
 P 5200 3150
-F 0 "#PWR6" H 5200 3150 30  0001 C CNN
+F 0 "#PWR017" H 5200 3150 30  0001 C CNN
 F 1 "GND" H 5200 3080 30  0001 C CNN
 F 2 "" H 5200 3150 60  0000 C CNN
@@
 LCD-RS
 $Comp
-L GND #PWR7
+L GND #PWR018
 U 1 1 53EC1C74
 P 5200 3250
-F 0 "#PWR7" H 5200 3250 30  0001 C CNN
+F 0 "#PWR018" H 5200 3250 30  0001 C CNN
 F 1 "GND" H 5200 3180 30  0001 C CNN
 F 2 "" H 5200 3250 60  0000 C CNN
@@
 LCD-D3
 $Comp
-L GND #PWR10
+L GND #PWR019
 U 1 1 53EC1E47
 P 6000 4800
-F 0 "#PWR10" H 6000 4800 30  0001 C CNN
+F 0 "#PWR019" H 6000 4800 30  0001 C CNN
 F 1 "GND" H 6000 4730 30  0001 C CNN
 F 2 "" H 6000 4800 60  0000 C CNN
@@
 	4450 2150 5250 2150
 $Comp
-L GND #PWR11
+L GND #PWR020
 U 1 1 53EC2288
 P 6850 3500
-F 0 "#PWR11" H 6850 3500 30  0001 C CNN
+F 0 "#PWR020" H 6850 3500 30  0001 C CNN
 F 1 "GND" H 6850 3430 30  0001 C CNN
 F 2 "" H 6850 3500 60  0000 C CNN
@@
 	9350 3400 9200 3400
 $Comp
-L GND #PWR19
+L GND #PWR021
 U 1 1 53EC2456
 P 9150 3450
-F 0 "#PWR19" H 9150 3450 30  0001 C CNN
+F 0 "#PWR021" H 9150 3450 30  0001 C CNN
 F 1 "GND" H 9150 3380 30  0001 C CNN
 F 2 "" H 9150 3450 60  0000 C CNN
@@
 F 0 "P1" V 4950 1550 50  0000 C CNN
 F 1 "Prog" V 5050 1550 50  0000 C CNN
-F 2 "" H 5000 1550 60  0000 C CNN
+F 2 "Connect:SIL-5" H 5000 1550 60  0000 C CNN
 F 3 "" H 5000 1550 60  0000 C CNN
 	1    5000 1550
@@
 $EndComp
 $Comp
-L GND #PWR3
+L GND #PWR022
 U 1 1 53ECE752
 P 4600 1800
-F 0 "#PWR3" H 4600 1800 30  0001 C CNN
+F 0 "#PWR022" H 4600 1800 30  0001 C CNN
 F 1 "GND" H 4600 1730 30  0001 C CNN
 F 2 "" H 4600 1800 60  0000 C CNN
@@
 F 0 "R1" V 4930 2500 50  0000 C CNN
 F 1 "2.2k" V 4850 2500 50  0000 C CNN
-F 2 "" H 4850 2500 60  0000 C CNN
+F 2 "SMD_Packages:SMD-0805" H 4850 2500 60  0000 C CNN
 F 3 "" H 4850 2500 60  0000 C CNN
 	1    4850 2500
@@
 RX
 $Comp
-L GND #PWR?
+L GND #PWR023
 U 1 1 53ED5509
 P 8700 3500
-F 0 "#PWR?" H 8700 3500 30  0001 C CNN
+F 0 "#PWR023" H 8700 3500 30  0001 C CNN
 F 1 "GND" H 8700 3430 30  0001 C CNN
 F 2 "" H 8700 3500 60  0000 C CNN
