File: hardware/terminal/terminal.sch (KiCad schematic (older format))
At the start: 14 parts, among them IC1 ATMEGA8-P, J1 RJ45, P1 Prog, P2 RC522, P3 LCD, P4 Keypad, U1 7805, U2 MAX232, U3 7803

Commit message: o Basic placement.
Connections:
- net labels added: RX-ext, TX-ext
Changed lines of the file:
@@
 LIBS:valves
 LIBS:xilinx
-LIBS:terminal-cache
 EELAYER 24 0
 EELAYER END
@@
 Text GLabel 4050 3600 2    50   Output ~ 0
 TX
-$Comp
-L +12V #PWR03
-U 1 1 53EB8601
-P 8800 3700
-F 0 "#PWR03" H 8800 3650 20  0001 C CNN
-F 1 "+12V" H 8800 3800 30  0000 C CNN
-F 2 "" H 8800 3700 60  0000 C CNN
-F 3 "" H 8800 3700 60  0000 C CNN
-	1    8800 3700
-	1    0    0    -1
-$EndComp
 Wire Wire Line
 	8800 3700 9350 3700
@@
 $EndComp
 $Comp
-L GND #PWR04
+L GND #PWR03
 U 1 1 53EB881B
 P 10150 4000
-F 0 "#PWR04" H 10150 4000 30  0001 C CNN
+F 0 "#PWR03" H 10150 4000 30  0001 C CNN
 F 1 "GND" H 10150 3930 30  0001 C CNN
 F 2 "" H 10150 4000 60  0000 C CNN
@@
 	1    0    0    -1
 $EndComp
-$Comp
-L +12V #PWR05
-U 1 1 53EB882F
-P 8600 4100
-F 0 "#PWR05" H 8600 4050 20  0001 C CNN
-F 1 "+12V" H 8600 4200 30  0000 C CNN
-F 2 "" H 8600 4100 60  0000 C CNN
-F 3 "" H 8600 4100 60  0000 C CNN
-	1    8600 4100
-	1    0    0    -1
-$EndComp
 Wire Wire Line
 	8600 4100 8600 4150
 $Comp
-L GND #PWR06
+L GND #PWR04
 U 1 1 53EB884F
 P 9000 4450
-F 0 "#PWR06" H 9000 4450 30  0001 C CNN
+F 0 "#PWR04" H 9000 4450 30  0001 C CNN
 F 1 "GND" H 9000 4380 30  0001 C CNN
 F 2 "" H 9000 4450 60  0000 C CNN
@@
 $EndComp
 $Comp
-L +3.3V #PWR07
+L +3.3V #PWR05
 U 1 1 53EB8966
 P 9400 4100
-F 0 "#PWR07" H 9400 4060 30  0001 C CNN
+F 0 "#PWR05" H 9400 4060 30  0001 C CNN
 F 1 "+3.3V" H 9400 4210 30  0000 C CNN
 F 2 "" H 9400 4100 60  0000 C CNN
@@
 	9400 4150 9400 4100
 $Comp
-L +3.3V #PWR08
+L +3.3V #PWR06
 U 1 1 53EB89B2
 P 5250 2000
-F 0 "#PWR08" H 5250 1960 30  0001 C CNN
+F 0 "#PWR06" H 5250 1960 30  0001 C CNN
 F 1 "+3.3V" H 5250 2110 30  0000 C CNN
 F 2 "" H 5250 2000 60  0000 C CNN
@@
 	4050 2200 4450 2200
 $Comp
-L GND #PWR09
+L GND #PWR07
 U 1 1 53EB89F8
 P 5100 2300
-F 0 "#PWR09" H 5100 2300 30  0001 C CNN
+F 0 "#PWR07" H 5100 2300 30  0001 C CNN
 F 1 "GND" H 5100 2230 30  0001 C CNN
 F 2 "" H 5100 2300 60  0000 C CNN
@@
 $EndComp
 $Comp
-L GND #PWR010
+L GND #PWR08
 U 1 1 53EB8B64
 P 3050 4700
-F 0 "#PWR010" H 3050 4700 30  0001 C CNN
+F 0 "#PWR08" H 3050 4700 30  0001 C CNN
 F 1 "GND" H 3050 4630 30  0001 C CNN
 F 2 "" H 3050 4700 60  0000 C CNN
@@
 $EndComp
 $Comp
-L +3.3V #PWR011
+L +3.3V #PWR09
 U 1 1 53EB8B76
 P 3050 1800
-F 0 "#PWR011" H 3050 1760 30  0001 C CNN
+F 0 "#PWR09" H 3050 1760 30  0001 C CNN
 F 1 "+3.3V" H 3050 1910 30  0000 C CNN
 F 2 "" H 3050 1800 60  0000 C CNN
@@
 $EndComp
 $Comp
-L +12V #PWR012
+L +12V #PWR010
 U 1 1 53EC1B72
 P 7350 4100
-F 0 "#PWR012" H 7350 4050 20  0001 C CNN
+F 0 "#PWR010" H 7350 4050 20  0001 C CNN
 F 1 "+12V" H 7350 4200 30  0000 C CNN
 F 2 "" H 7350 4100 60  0000 C CNN
@@
 	7350 4100 7350 4150
 $Comp
-L +5V #PWR013
+L +5V #PWR011
 U 1 1 53EC1BA0
 P 8150 4100
-F 0 "#PWR013" H 8150 4190 20  0001 C CNN
+F 0 "#PWR011" H 8150 4190 20  0001 C CNN
 F 1 "+5V" H 8150 4190 30  0000 C CNN
 F 2 "" H 8150 4100 60  0000 C CNN
@@
 	8150 4100 8150 4150
 $Comp
-L GND #PWR014
+L GND #PWR012
 U 1 1 53EC1BD4
 P 7750 4450
-F 0 "#PWR014" H 7750 4450 30  0001 C CNN
+F 0 "#PWR012" H 7750 4450 30  0001 C CNN
 F 1 "GND" H 7750 4380 30  0001 C CNN
 F 2 "" H 7750 4450 60  0000 C CNN
@@
 $EndComp
 $Comp
-L GND #PWR015
+L GND #PWR013
 U 1 1 53EC1BE1
 P 5200 3050
-F 0 "#PWR015" H 5200 3050 30  0001 C CNN
+F 0 "#PWR013" H 5200 3050 30  0001 C CNN
 F 1 "GND" H 5200 2980 30  0001 C CNN
 F 2 "" H 5200 3050 60  0000 C CNN
@@
 $EndComp
 $Comp
-L +5V #PWR016
+L +5V #PWR014
 U 1 1 53EC1BF5
 P 6000 3050
-F 0 "#PWR016" H 6000 3140 20  0001 C CNN
+F 0 "#PWR014" H 6000 3140 20  0001 C CNN
 F 1 "+5V" H 6000 3140 30  0000 C CNN
 F 2 "" H 6000 3050 60  0000 C CNN
@@
 $EndComp
 $Comp
-L GND #PWR017
+L GND #PWR015
 U 1 1 53EC1C07
 P 5200 3150
-F 0 "#PWR017" H 5200 3150 30  0001 C CNN
+F 0 "#PWR015" H 5200 3150 30  0001 C CNN
 F 1 "GND" H 5200 3080 30  0001 C CNN
 F 2 "" H 5200 3150 60  0000 C CNN
@@
 LCD-RS
 $Comp
-L GND #PWR018
+L GND #PWR016
 U 1 1 53EC1C74
 P 5200 3250
-F 0 "#PWR018" H 5200 3250 30  0001 C CNN
+F 0 "#PWR016" H 5200 3250 30  0001 C CNN
 F 1 "GND" H 5200 3180 30  0001 C CNN
 F 2 "" H 5200 3250 60  0000 C CNN
@@
 LCD-D3
 $Comp
-L GND #PWR019
+L GND #PWR017
 U 1 1 53EC1E47
 P 6000 4800
-F 0 "#PWR019" H 6000 4800 30  0001 C CNN
+F 0 "#PWR017" H 6000 4800 30  0001 C CNN
 F 1 "GND" H 6000 4730 30  0001 C CNN
 F 2 "" H 6000 4800 60  0000 C CNN
@@
 Text GLabel 4050 4200 2    50   Output ~ 0
 KROW-3
-Text GLabel 5200 4000 0    50   Input ~ 0
+Text GLabel 5200 4700 0    50   Input ~ 0
 KROW-0
+Text GLabel 5200 4600 0    50   Input ~ 0
+KROW-1
+Text GLabel 5200 4500 0    50   Input ~ 0
+KROW-2
+Text GLabel 5200 4400 0    50   Input ~ 0
+KROW-3
+Text GLabel 5200 4300 0    50   Input ~ 0
+KCOL-0
+Text GLabel 5200 4200 0    50   Input ~ 0
+KCOL-1
 Text GLabel 5200 4100 0    50   Input ~ 0
-KROW-1
-Text GLabel 5200 4200 0    50   Input ~ 0
-KROW-2
-Text GLabel 5200 4300 0    50   Input ~ 0
-KROW-3
-Text GLabel 5200 4400 0    50   Input ~ 0
-KCOL-0
-Text GLabel 5200 4500 0    50   Input ~ 0
-KCOL-1
-Text GLabel 5200 4600 0    50   Input ~ 0
 KCOL-2
 Wire Wire Line
@@
 	4450 2150 5250 2150
 $Comp
-L GND #PWR020
+L GND #PWR018
 U 1 1 53EC2288
 P 6850 3500
-F 0 "#PWR020" H 6850 3500 30  0001 C CNN
+F 0 "#PWR018" H 6850 3500 30  0001 C CNN
 F 1 "GND" H 6850 3430 30  0001 C CNN
 F 2 "" H 6850 3500 60  0000 C CNN
@@
 	9350 3400 9200 3400
 $Comp
-L GND #PWR021
+L GND #PWR019
 U 1 1 53EC2456
 P 9150 3450
-F 0 "#PWR021" H 9150 3450 30  0001 C CNN
+F 0 "#PWR019" H 9150 3450 30  0001 C CNN
 F 1 "GND" H 9150 3380 30  0001 C CNN
 F 2 "" H 9150 3450 60  0000 C CNN
@@
 $EndComp
 $Comp
-L GND #PWR022
+L GND #PWR020
 U 1 1 53ECE752
 P 4600 1800
-F 0 "#PWR022" H 4600 1800 30  0001 C CNN
+F 0 "#PWR020" H 4600 1800 30  0001 C CNN
 F 1 "GND" H 4600 1730 30  0001 C CNN
 F 2 "" H 4600 1800 60  0000 C CNN
@@
 RX
 $Comp
-L GND #PWR023
+L GND #PWR021
 U 1 1 53ED5509
 P 8700 3500
-F 0 "#PWR023" H 8700 3500 30  0001 C CNN
+F 0 "#PWR021" H 8700 3500 30  0001 C CNN
 F 1 "GND" H 8700 3430 30  0001 C CNN
 F 2 "" H 8700 3500 60  0000 C CNN
@@
 Wire Wire Line
 	8700 3400 8700 3500
+Connection ~ 4850 2750
+$Comp
+L +12V #PWR022
+U 1 1 53EE3255
+P 8800 3700
+F 0 "#PWR022" H 8800 3650 20  0001 C CNN
+F 1 "+12V" H 8800 3800 30  0000 C CNN
+F 2 "" H 8800 3700 60  0000 C CNN
+F 3 "" H 8800 3700 60  0000 C CNN
+	1    8800 3700
+	1    0    0    -1
+$EndComp
+$Comp
+L +12V #PWR023
+U 1 1 53EE5EAC
+P 8600 4100
+F 0 "#PWR023" H 8600 4050 20  0001 C CNN
+F 1 "+12V" H 8600 4200 30  0000 C CNN
+F 2 "" H 8600 4100 60  0000 C CNN
+F 3 "" H 8600 4100 60  0000 C CNN
+	1    8600 4100
+	1    0    0    -1
+$EndComp
+Text Label 8950 3100 0    60   ~ 0
+TX-ext
+Text Label 9050 3600 0    60   ~ 0
+RX-ext
 $EndSCHEMATC

Commit message: Work in progress  o more layout work done  o use chargepump of remaining rs232 driver to provide negative    voltage to display.
Parts:
- removed U1: 7805, Discret:LM78XXV, symbol 7805
- added C5, C6: C, Capacitors_SMD:c_0805, symbol C
- added P10: CONN_4, Connect:SIL-4, symbol CONN_4
- added P5, P6, P7, P8: CONN_1, Connect:1pin, symbol CONN_1
- added P9: CONN_2X2, Pin_Headers:Pin_Header_Straight_2x02, symbol CONN_2X2
- added R2: 2.2k, SMD_Packages:SM0805, symbol R
- added R3, R4: 82, SMD_Packages:SM0805, symbol R
- U2: value MAX232 -> SP3232E
Connections:
- net labels added: CS-RFID, LCD-contr, RST-RFID
- wire segments 41 -> 52
Other:
- moved on the sheet: U3

Commit message: o add voltage divider LCD contrast.
Parts:
- added R?: 3k, SMD_Packages:SMD-0805, symbol R
- added R?: 2.2k, SMD_Packages:SMD-0805, symbol R
Connections:
- wire segments 52 -> 59
Changed lines of the file:
@@
 L CONN_8X2 P3
 U 1 1 53EB8E37
-P 5600 3400
-F 0 "P3" H 5600 3850 60  0000 C CNN
-F 1 "LCD" V 5600 3400 50  0000 C CNN
-F 2 "Pin_Headers:Pin_Header_Straight_2x08" H 5600 3400 60  0000 C CNN
-F 3 "" H 5600 3400 60  0000 C CNN
-	1    5600 3400
+P 5600 3350
+F 0 "P3" H 5600 3800 60  0000 C CNN
+F 1 "LCD" V 5600 3350 50  0000 C CNN
+F 2 "Pin_Headers:Pin_Header_Straight_2x08" H 5600 3350 60  0000 C CNN
+F 3 "" H 5600 3350 60  0000 C CNN
+	1    5600 3350
 	1    0    0    -1
 $EndComp
@@
 L GND #PWR010
 U 1 1 53EC1BE1
-P 5200 3050
-F 0 "#PWR010" H 5200 3050 30  0001 C CNN
-F 1 "GND" H 5200 2980 30  0001 C CNN
-F 2 "" H 5200 3050 60  0000 C CNN
-F 3 "" H 5200 3050 60  0000 C CNN
-	1    5200 3050
+P 5200 3000
+F 0 "#PWR010" H 5200 3000 30  0001 C CNN
+F 1 "GND" H 5200 2930 30  0001 C CNN
+F 2 "" H 5200 3000 60  0000 C CNN
+F 3 "" H 5200 3000 60  0000 C CNN
+	1    5200 3000
 	0    1    1    0
 $EndComp
@@
 L +5V #PWR011
 U 1 1 53EC1BF5
-P 6000 3050
-F 0 "#PWR011" H 6000 3140 20  0001 C CNN
-F 1 "+5V" H 6000 3140 30  0000 C CNN
-F 2 "" H 6000 3050 60  0000 C CNN
-F 3 "" H 6000 3050 60  0000 C CNN
-	1    6000 3050
+P 6000 3000
+F 0 "#PWR011" H 6000 3090 20  0001 C CNN
+F 1 "+5V" H 6000 3090 30  0000 C CNN
+F 2 "" H 6000 3000 60  0000 C CNN
+F 3 "" H 6000 3000 60  0000 C CNN
+	1    6000 3000
 	0    1    1    0
 $EndComp
@@
 L GND #PWR012
 U 1 1 53EC1C74
-P 5200 3250
-F 0 "#PWR012" H 5200 3250 30  0001 C CNN
-F 1 "GND" H 5200 3180 30  0001 C CNN
-F 2 "" H 5200 3250 60  0000 C CNN
-F 3 "" H 5200 3250 60  0000 C CNN
-	1    5200 3250
-	0    1    1    0
-$EndComp
-Text GLabel 6000 3150 2    50   Input ~ 0
+P 5200 3200
+F 0 "#PWR012" H 5200 3200 30  0001 C CNN
+F 1 "GND" H 5200 3130 30  0001 C CNN
+F 2 "" H 5200 3200 60  0000 C CNN
+F 3 "" H 5200 3200 60  0000 C CNN
+	1    5200 3200
+	0    1    1    0
+$EndComp
+Text GLabel 6000 3100 2    50   Input ~ 0
 LCD-RS
 Text GLabel 4050 3300 2    50   Output ~ 0
 LCD-EN
-Text GLabel 6000 3250 2    50   Input ~ 0
+Text GLabel 6000 3200 2    50   Input ~ 0
 LCD-EN
 Text GLabel 4050 2800 2    50   Output ~ 0
@@
 Text GLabel 4050 3100 2    50   Output ~ 0
 LCD-D3
-Text GLabel 5200 3550 0    50   Input ~ 0
+Text GLabel 5200 3500 0    50   Input ~ 0
 LCD-D0
-Text GLabel 5200 3650 0    50   Input ~ 0
+Text GLabel 5200 3600 0    50   Input ~ 0
 LCD-D2
-Text GLabel 6000 3550 2    50   Input ~ 0
+Text GLabel 6000 3500 2    50   Input ~ 0
 LCD-D1
-Text GLabel 6000 3650 2    50   Input ~ 0
+Text GLabel 6000 3600 2    50   Input ~ 0
 LCD-D3
 $Comp
@@
 Text Label 4350 2300 0    60   ~ 0
 CS-RFID
-Text GLabel 5200 3150 0    50   Input ~ 0
+Text GLabel 6450 2750 0    50   Input ~ 0
 LCD-contr
 Text GLabel 8700 3200 2    50   Output ~ 0
@@
 Wire Wire Line
 	6800 3200 7100 3200
+$Comp
+L R R?
+U 1 1 53F0145B
+P 6200 2400
+F 0 "R?" V 6280 2400 50  0000 C CNN
+F 1 "3k" V 6200 2400 50  0000 C CNN
+F 2 "SMD_Packages:SMD-0805" H 6200 2400 60  0000 C CNN
+F 3 "" H 6200 2400 60  0000 C CNN
+	1    6200 2400
+	0    -1   1    0
+$EndComp
+$Comp
+L R R?
+U 1 1 53F015C0
+P 6200 2600
+F 0 "R?" V 6280 2600 50  0000 C CNN
+F 1 "2.2k" V 6200 2600 50  0000 C CNN
+F 2 "SMD_Packages:SMD-0805" H 6200 2600 60  0000 C CNN
+F 3 "" H 6200 2600 60  0000 C CNN
+	1    6200 2600
+	0    -1   1    0
+$EndComp
+$Comp
+L GND #PWR?
+U 1 1 53F01757
+P 6450 2400
+F 0 "#PWR?" H 6450 2400 30  0001 C CNN
+F 1 "GND" H 6450 2330 30  0001 C CNN
+F 2 "" H 6450 2400 60  0000 C CNN
+F 3 "" H 6450 2400 60  0000 C CNN
+	1    6450 2400
+	0    -1   1    0
+$EndComp
+Wire Wire Line
+	5950 2400 5950 2600
+Wire Wire Line
+	6450 2600 6450 2750
+Connection ~ 5950 2500
+Wire Wire Line
+	5950 2500 5850 2500
+Wire Wire Line
+	5850 2500 5850 2850
+Wire Wire Line
+	5850 2850 5050 2850
+Wire Wire Line
+	5050 2850 5050 3100
+Wire Wire Line
+	5050 3100 5200 3100
 $EndSCHEMATC

Commit message: o First complete routing. o Add voltage divider to get a proper negative voltage for LCD.
Parts:
- gave numbers to parts that had none: 2
Connections:
- net labels removed: +5V

Commit message: o Add 'playground' area.
Parts:
- added P11, P14: CONN_5X2, Pin_Headers:Pin_Header_Straight_2x05, symbol CONN_5X2
- added P12: CONN_4, Connect:SIL-4, symbol CONN_4
- added P13: CONN_3X2, Pin_Headers:Pin_Header_Straight_2x03, symbol CONN_3X2
Other:
- note added: "Playground Area"
Changed lines of the file:
@@
 $EndComp
 $Comp
-L GND #PWR01
+L GND #PWR22
 U 1 1 53EB83C0
 P 9250 2700
-F 0 "#PWR01" H 9250 2700 30  0001 C CNN
+F 0 "#PWR22" H 9250 2700 30  0001 C CNN
 F 1 "GND" H 9250 2630 30  0001 C CNN
 F 2 "" H 9250 2700 60  0001 C CNN
@@
 	7000 2900 7100 2900
 $Comp
-L +3.3V #PWR02
+L +3.3V #PWR18
 U 1 1 53EB841D
 P 8750 2000
-F 0 "#PWR02" H 8750 1960 30  0001 C CNN
+F 0 "#PWR18" H 8750 1960 30  0001 C CNN
 F 1 "+3.3V" H 8750 2110 30  0000 C CNN
 F 2 "" H 8750 2000 60  0001 C CNN
@@
 $EndComp
 $Comp
-L GND #PWR03
+L GND #PWR26
 U 1 1 53EB881B
 P 10150 4000
-F 0 "#PWR03" H 10150 4000 30  0001 C CNN
+F 0 "#PWR26" H 10150 4000 30  0001 C CNN
 F 1 "GND" H 10150 3930 30  0001 C CNN
 F 2 "" H 10150 4000 60  0001 C CNN
@@
 	8450 4050 8450 4100
 $Comp
-L GND #PWR04
+L GND #PWR20
 U 1 1 53EB884F
 P 8850 4400
-F 0 "#PWR04" H 8850 4400 30  0001 C CNN
+F 0 "#PWR20" H 8850 4400 30  0001 C CNN
 F 1 "GND" H 8850 4330 30  0001 C CNN
 F 2 "" H 8850 4400 60  0001 C CNN
@@
 $EndComp
 $Comp
-L +3.3V #PWR05
+L +3.3V #PWR23
 U 1 1 53EB8966
 P 9250 4050
-F 0 "#PWR05" H 9250 4010 30  0001 C CNN
+F 0 "#PWR23" H 9250 4010 30  0001 C CNN
 F 1 "+3.3V" H 9250 4160 30  0000 C CNN
 F 2 "" H 9250 4050 60  0001 C CNN
@@
 	9250 4100 9250 4050
 $Comp
-L +3.3V #PWR06
+L +3.3V #PWR9
 U 1 1 53EB89B2
 P 5250 2000
-F 0 "#PWR06" H 5250 1960 30  0001 C CNN
+F 0 "#PWR9" H 5250 1960 30  0001 C CNN
 F 1 "+3.3V" H 5250 2110 30  0000 C CNN
 F 2 "" H 5250 2000 60  0001 C CNN
@@
 	4050 2200 4450 2200
 $Comp
-L GND #PWR07
+L GND #PWR6
 U 1 1 53EB89F8
 P 5100 2300
-F 0 "#PWR07" H 5100 2300 30  0001 C CNN
+F 0 "#PWR6" H 5100 2300 30  0001 C CNN
 F 1 "GND" H 5100 2230 30  0001 C CNN
 F 2 "" H 5100 2300 60  0001 C CNN
@@
 $EndComp
 $Comp
-L GND #PWR08
+L GND #PWR2
 U 1 1 53EB8B64
 P 3050 4700
-F 0 "#PWR08" H 3050 4700 30  0001 C CNN
+F 0 "#PWR2" H 3050 4700 30  0001 C CNN
 F 1 "GND" H 3050 4630 30  0001 C CNN
 F 2 "" H 3050 4700 60  0001 C CNN
@@
 $EndComp
 $Comp
-L +3.3V #PWR09
+L +3.3V #PWR1
 U 1 1 53EB8B76
 P 3050 1800
-F 0 "#PWR09" H 3050 1760 30  0001 C CNN
+F 0 "#PWR1" H 3050 1760 30  0001 C CNN
 F 1 "+3.3V" H 3050 1910 30  0000 C CNN
 F 2 "" H 3050 1800 60  0001 C CNN
@@
 $EndComp
 $Comp
-L GND #PWR010
+L GND #PWR7
 U 1 1 53EC1BE1
 P 5200 3000
-F 0 "#PWR010" H 5200 3000 30  0001 C CNN
+F 0 "#PWR7" H 5200 3000 30  0001 C CNN
 F 1 "GND" H 5200 2930 30  0001 C CNN
 F 2 "" H 5200 3000 60  0001 C CNN
@@
 LCD-RS
 $Comp
-L GND #PWR011
+L GND #PWR8
 U 1 1 53EC1C74
 P 5200 3200
-F 0 "#PWR011" H 5200 3200 30  0001 C CNN
+F 0 "#PWR8" H 5200 3200 30  0001 C CNN
 F 1 "GND" H 5200 3130 30  0001 C CNN
 F 2 "" H 5200 3200 60  0001 C CNN
@@
 LCD-D3
 $Comp
-L GND #PWR012
+L GND #PWR11
 U 1 1 53EC1E47
 P 6000 4800
-F 0 "#PWR012" H 6000 4800 30  0001 C CNN
+F 0 "#PWR11" H 6000 4800 30  0001 C CNN
 F 1 "GND" H 6000 4730 30  0001 C CNN
 F 2 "" H 6000 4800 60  0001 C CNN
@@
 	9350 3400 9200 3400
 $Comp
-L GND #PWR013
+L GND #PWR21
 U 1 1 53EC2456
 P 9150 3450
-F 0 "#PWR013" H 9150 3450 30  0001 C CNN
+F 0 "#PWR21" H 9150 3450 30  0001 C CNN
 F 1 "GND" H 9150 3380 30  0001 C CNN
 F 2 "" H 9150 3450 60  0001 C CNN
@@
 $EndComp
 $Comp
-L GND #PWR014
+L GND #PWR4
 U 1 1 53ECE752
 P 4600 1800
-F 0 "#PWR014" H 4600 1800 30  0001 C CNN
+F 0 "#PWR4" H 4600 1800 30  0001 C CNN
 F 1 "GND" H 4600 1730 30  0001 C CNN
 F 2 "" H 4600 1800 60  0001 C CNN
@@
 RX
 $Comp
-L GND #PWR015
+L GND #PWR17
 U 1 1 53ED5509
 P 8700 3500
-F 0 "#PWR015" H 8700 3500 30  0001 C CNN
+F 0 "#PWR17" H 8700 3500 30  0001 C CNN
 F 1 "GND" H 8700 3430 30  0001 C CNN
 F 2 "" H 8700 3500 60  0001 C CNN
@@
 Connection ~ 4850 2750
 $Comp
-L +12V #PWR016
+L +12V #PWR19
 U 1 1 53EE3255
 P 8800 3700
-F 0 "#PWR016" H 8800 3650 20  0001 C CNN
+F 0 "#PWR19" H 8800 3650 20  0001 C CNN
 F 1 "+12V" H 8800 3800 30  0000 C CNN
 F 2 "" H 8800 3700 60  0001 C CNN
@@
 $EndComp
 $Comp
-L +12V #PWR017
+L +12V #PWR16
 U 1 1 53EE5EAC
 P 8450 4050
-F 0 "#PWR017" H 8450 4000 20  0001 C CNN
+F 0 "#PWR16" H 8450 4000 20  0001 C CNN
 F 1 "+12V" H 8450 4150 30  0000 C CNN
 F 2 "" H 8450 4050 60  0001 C CNN
@@
 Connection ~ 3650 1350
 $Comp
-L +3.3V #PWR018
+L +3.3V #PWR3
 U 1 1 53EEF690
 P 4150 1150
-F 0 "#PWR018" H 4150 1110 30  0001 C CNN
+F 0 "#PWR3" H 4150 1110 30  0001 C CNN
 F 1 "+3.3V" H 4150 1260 30  0000 C CNN
 F 2 "" H 4150 1150 60  0001 C CNN
@@
 	4600 4650 4700 4650
 $Comp
-L GND #PWR019
+L GND #PWR5
 U 1 1 53EF0029
 P 4650 4750
-F 0 "#PWR019" H 4650 4750 30  0001 C CNN
+F 0 "#PWR5" H 4650 4750 30  0001 C CNN
 F 1 "GND" H 4650 4680 30  0001 C CNN
 F 2 "" H 4650 4750 60  0001 C CNN
@@
 $EndComp
 $Comp
-L GND #PWR020
+L GND #PWR25
 U 1 1 53EF055A
 P 9750 2450
-F 0 "#PWR020" H 9750 2450 30  0001 C CNN
+F 0 "#PWR25" H 9750 2450 30  0001 C CNN
 F 1 "GND" H 9750 2380 30  0001 C CNN
 F 2 "" H 9750 2450 60  0001 C CNN
@@
 	9750 2400 9750 2450
 $Comp
-L +12V #PWR021
+L +12V #PWR24
 U 1 1 53EF05EE
 P 9750 2050
-F 0 "#PWR021" H 9750 2000 20  0001 C CNN
+F 0 "#PWR24" H 9750 2000 20  0001 C CNN
 F 1 "+12V" H 9750 2150 30  0000 C CNN
 F 2 "" H 9750 2050 60  0001 C CNN
@@
 $EndComp
 $Comp
-L GND #PWR022
+L GND #PWR15
 U 1 1 53EF7CD3
 P 7800 4450
-F 0 "#PWR022" H 7800 4450 30  0001 C CNN
+F 0 "#PWR15" H 7800 4450 30  0001 C CNN
 F 1 "GND" H 7800 4380 30  0001 C CNN
 F 2 "" H 7800 4450 60  0001 C CNN
@@
 	7650 4000 7950 4000
 $Comp
-L +3.3V #PWR023
+L +3.3V #PWR14
 U 1 1 53EF7E3C
 P 7800 3950
-F 0 "#PWR023" H 7800 3910 30  0001 C CNN
+F 0 "#PWR14" H 7800 3910 30  0001 C CNN
 F 1 "+3.3V" H 7800 4060 30  0000 C CNN
 F 2 "" H 7800 3950 60  0001 C CNN
@@
 LCD-contr
 $Comp
-L +3.3V #PWR024
+L +3.3V #PWR13
 U 1 1 53EFB331
 P 6800 3200
-F 0 "#PWR024" H 6800 3160 30  0001 C CNN
+F 0 "#PWR13" H 6800 3160 30  0001 C CNN
 F 1 "+3.3V" H 6800 3310 30  0000 C CNN
 F 2 "" H 6800 3200 60  0001 C CNN
@@
 $EndComp
 $Comp
-L GND #PWR025
+L GND #PWR12
 U 1 1 53F01757
 P 6450 2400
-F 0 "#PWR025" H 6450 2400 30  0001 C CNN
+F 0 "#PWR12" H 6450 2400 30  0001 C CNN
 F 1 "GND" H 6450 2330 30  0001 C CNN
 F 2 "" H 6450 2400 60  0001 C CNN
@@
 	5050 3100 5200 3100
 $Comp
-L +3.3V #PWR026
+L +3.3V #PWR10
 U 1 1 53F0185A
 P 6000 3000
-F 0 "#PWR026" H 6000 2960 30  0001 C CNN
+F 0 "#PWR10" H 6000 2960 30  0001 C CNN
 F 1 "+3.3V" H 6000 3110 30  0000 C CNN
 F 2 "" H 6000 3000 60  0001 C CNN
@@
 	0    1    1    0
 $EndComp
+$Comp
+L CONN_5X2 P11
+U 1 1 53F031B7
+P 3250 5550
+F 0 "P11" H 3250 5850 60  0000 C CNN
+F 1 "CONN_5X2" V 3250 5550 50  0000 C CNN
+F 2 "Pin_Headers:Pin_Header_Straight_2x05" H 3250 5550 60  0001 C CNN
+F 3 "" H 3250 5550 60  0000 C CNN
+	1    3250 5550
+	1    0    0    -1
+$EndComp
+$Comp
+L CONN_5X2 P14
+U 1 1 53F03214
+P 4200 5550
+F 0 "P14" H 4200 5850 60  0000 C CNN
+F 1 "CONN_5X2" V 4200 5550 50  0000 C CNN
+F 2 "Pin_Headers:Pin_Header_Straight_2x05" H 4200 5550 60  0001 C CNN
+F 3 "" H 4200 5550 60  0000 C CNN
+	1    4200 5550
+	1    0    0    -1
+$EndComp
+$Comp
+L CONN_4 P12
+U 1 1 53F03279
+P 3250 6100
+F 0 "P12" V 3200 6100 50  0000 C CNN
+F 1 "CONN_4" V 3300 6100 50  0000 C CNN
+F 2 "Connect:SIL-4" H 3250 6100 60  0001 C CNN
+F 3 "" H 3250 6100 60  0000 C CNN
+	1    3250 6100
+	1    0    0    -1
+$EndComp
+$Comp
+L CONN_3X2 P13
+U 1 1 53F0330C
+P 4000 6150
+F 0 "P13" H 4000 6400 50  0000 C CNN
+F 1 "CONN_3X2" V 4000 6200 40  0000 C CNN
+F 2 "Pin_Headers:Pin_Header_Straight_2x03" H 4000 6150 60  0001 C CNN
+F 3 "" H 4000 6150 60  0000 C CNN
+	1    4000 6150
+	1    0    0    -1
+$EndComp
+Text Notes 2600 5150 0    60   ~ 0
+Playground Area
 $EndSCHEMATC
