File: hardware/terminal/terminal.sch (KiCad schematic (older format))
At the start: 33 parts, among them IC1 ATMEGA8-P, J1 RJ45, P1 Prog, P10 CONN_4, P11 CONN_5X2, P12 CONN_4, P13 CONN_3X2, P14 CONN_5X2, P2 RC522, P3 LCD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

Commit message: o anothe de-coupling capacitor close to the SP3232E can't harm.
Parts:
- added C9: C, Capacitors_SMD:c_0805, symbol C
Changed lines of the file:
@@
 $EndComp
 $Comp
-L GND #PWR01
+L GND #PWR24
 U 1 1 53EB83C0
 P 9250 2700
-F 0 "#PWR01" H 9250 2700 30  0001 C CNN
+F 0 "#PWR24" H 9250 2700 30  0001 C CNN
 F 1 "GND" H 9250 2630 30  0001 C CNN
 F 2 "" H 9250 2700 60  0001 C CNN
@@
 	7000 2900 7100 2900
 $Comp
-L +3.3V #PWR02
+L +3.3V #PWR20
 U 1 1 53EB841D
 P 8750 2000
-F 0 "#PWR02" H 8750 1960 30  0001 C CNN
+F 0 "#PWR20" H 8750 1960 30  0001 C CNN
 F 1 "+3.3V" H 8750 2110 30  0000 C CNN
 F 2 "" H 8750 2000 60  0001 C CNN
@@
 $EndComp
 $Comp
-L GND #PWR03
+L GND #PWR28
 U 1 1 53EB881B
 P 10150 4000
-F 0 "#PWR03" H 10150 4000 30  0001 C CNN
+F 0 "#PWR28" H 10150 4000 30  0001 C CNN
 F 1 "GND" H 10150 3930 30  0001 C CNN
 F 2 "" H 10150 4000 60  0001 C CNN
@@
 	8450 4050 8450 4100
 $Comp
-L GND #PWR04
+L GND #PWR22
 U 1 1 53EB884F
 P 8850 4550
-F 0 "#PWR04" H 8850 4550 30  0001 C CNN
+F 0 "#PWR22" H 8850 4550 30  0001 C CNN
 F 1 "GND" H 8850 4480 30  0001 C CNN
 F 2 "" H 8850 4550 60  0001 C CNN
@@
 $EndComp
 $Comp
-L +3.3V #PWR05
+L +3.3V #PWR25
 U 1 1 53EB8966
 P 9250 4050
-F 0 "#PWR05" H 9250 4010 30  0001 C CNN
+F 0 "#PWR25" H 9250 4010 30  0001 C CNN
 F 1 "+3.3V" H 9250 4160 30  0000 C CNN
 F 2 "" H 9250 4050 60  0001 C CNN
@@
 	9250 4100 9250 4050
 $Comp
-L +3.3V #PWR06
+L +3.3V #PWR9
 U 1 1 53EB89B2
 P 5250 2000
-F 0 "#PWR06" H 5250 1960 30  0001 C CNN
+F 0 "#PWR9" H 5250 1960 30  0001 C CNN
 F 1 "+3.3V" H 5250 2110 30  0000 C CNN
 F 2 "" H 5250 2000 60  0001 C CNN
@@
 	4050 2200 4450 2200
 $Comp
-L GND #PWR07
+L GND #PWR6
 U 1 1 53EB89F8
 P 5100 2300
-F 0 "#PWR07" H 5100 2300 30  0001 C CNN
+F 0 "#PWR6" H 5100 2300 30  0001 C CNN
 F 1 "GND" H 5100 2230 30  0001 C CNN
 F 2 "" H 5100 2300 60  0001 C CNN
@@
 $EndComp
 $Comp
-L GND #PWR08
+L GND #PWR2
 U 1 1 53EB8B64
 P 3050 4700
-F 0 "#PWR08" H 3050 4700 30  0001 C CNN
+F 0 "#PWR2" H 3050 4700 30  0001 C CNN
 F 1 "GND" H 3050 4630 30  0001 C CNN
 F 2 "" H 3050 4700 60  0001 C CNN
@@
 $EndComp
 $Comp
-L +3.3V #PWR09
+L +3.3V #PWR1
 U 1 1 53EB8B76
 P 3050 1800
-F 0 "#PWR09" H 3050 1760 30  0001 C CNN
+F 0 "#PWR1" H 3050 1760 30  0001 C CNN
 F 1 "+3.3V" H 3050 1910 30  0000 C CNN
 F 2 "" H 3050 1800 60  0001 C CNN
@@
 $EndComp
 $Comp
-L GND #PWR010
+L GND #PWR7
 U 1 1 53EC1BE1
 P 5200 3000
-F 0 "#PWR010" H 5200 3000 30  0001 C CNN
+F 0 "#PWR7" H 5200 3000 30  0001 C CNN
 F 1 "GND" H 5200 2930 30  0001 C CNN
 F 2 "" H 5200 3000 60  0001 C CNN
@@
 LCD-RS
 $Comp
-L GND #PWR011
+L GND #PWR8
 U 1 1 53EC1C74
 P 5200 3200
-F 0 "#PWR011" H 5200 3200 30  0001 C CNN
+F 0 "#PWR8" H 5200 3200 30  0001 C CNN
 F 1 "GND" H 5200 3130 30  0001 C CNN
 F 2 "" H 5200 3200 60  0001 C CNN
@@
 LCD-D3
 $Comp
-L GND #PWR012
+L GND #PWR11
 U 1 1 53EC1E47
 P 6000 4800
-F 0 "#PWR012" H 6000 4800 30  0001 C CNN
+F 0 "#PWR11" H 6000 4800 30  0001 C CNN
 F 1 "GND" H 6000 4730 30  0001 C CNN
 F 2 "" H 6000 4800 60  0001 C CNN
@@
 	9350 3400 9200 3400
 $Comp
-L GND #PWR013
+L GND #PWR23
 U 1 1 53EC2456
 P 9150 3450
-F 0 "#PWR013" H 9150 3450 30  0001 C CNN
+F 0 "#PWR23" H 9150 3450 30  0001 C CNN
 F 1 "GND" H 9150 3380 30  0001 C CNN
 F 2 "" H 9150 3450 60  0001 C CNN
@@
 $EndComp
 $Comp
-L GND #PWR014
+L GND #PWR4
 U 1 1 53ECE752
 P 4600 1800
-F 0 "#PWR014" H 4600 1800 30  0001 C CNN
+F 0 "#PWR4" H 4600 1800 30  0001 C CNN
 F 1 "GND" H 4600 1730 30  0001 C CNN
 F 2 "" H 4600 1800 60  0001 C CNN
@@
 RX
 $Comp
-L GND #PWR015
+L GND #PWR19
 U 1 1 53ED5509
 P 8700 3500
-F 0 "#PWR015" H 8700 3500 30  0001 C CNN
+F 0 "#PWR19" H 8700 3500 30  0001 C CNN
 F 1 "GND" H 8700 3430 30  0001 C CNN
 F 2 "" H 8700 3500 60  0001 C CNN
@@
 Connection ~ 4850 2750
 $Comp
-L +12V #PWR016
+L +12V #PWR21
 U 1 1 53EE3255
 P 8800 3700
-F 0 "#PWR016" H 8800 3650 20  0001 C CNN
+F 0 "#PWR21" H 8800 3650 20  0001 C CNN
 F 1 "+12V" H 8800 3800 30  0000 C CNN
 F 2 "" H 8800 3700 60  0001 C CNN
@@
 $EndComp
 $Comp
-L +12V #PWR017
+L +12V #PWR18
 U 1 1 53EE5EAC
 P 8450 4050
-F 0 "#PWR017" H 8450 4000 20  0001 C CNN
+F 0 "#PWR18" H 8450 4000 20  0001 C CNN
 F 1 "+12V" H 8450 4150 30  0000 C CNN
 F 2 "" H 8450 4050 60  0001 C CNN
@@
 Connection ~ 3650 1350
 $Comp
-L +3.3V #PWR018
+L +3.3V #PWR3
 U 1 1 53EEF690
 P 4150 1150
-F 0 "#PWR018" H 4150 1110 30  0001 C CNN
+F 0 "#PWR3" H 4150 1110 30  0001 C CNN
 F 1 "+3.3V" H 4150 1260 30  0000 C CNN
 F 2 "" H 4150 1150 60  0001 C CNN
@@
 	4600 4650 4700 4650
 $Comp
-L GND #PWR019
+L GND #PWR5
 U 1 1 53EF0029
 P 4650 4750
-F 0 "#PWR019" H 4650 4750 30  0001 C CNN
+F 0 "#PWR5" H 4650 4750 30  0001 C CNN
 F 1 "GND" H 4650 4680 30  0001 C CNN
 F 2 "" H 4650 4750 60  0001 C CNN
@@
 $EndComp
 $Comp
-L GND #PWR020
+L GND #PWR27
 U 1 1 53EF055A
 P 9750 2450
-F 0 "#PWR020" H 9750 2450 30  0001 C CNN
+F 0 "#PWR27" H 9750 2450 30  0001 C CNN
 F 1 "GND" H 9750 2380 30  0001 C CNN
 F 2 "" H 9750 2450 60  0001 C CNN
@@
 	9750 2400 9750 2450
 $Comp
-L +12V #PWR021
+L +12V #PWR26
 U 1 1 53EF05EE
 P 9750 2050
-F 0 "#PWR021" H 9750 2000 20  0001 C CNN
+F 0 "#PWR26" H 9750 2000 20  0001 C CNN
 F 1 "+12V" H 9750 2150 30  0000 C CNN
 F 2 "" H 9750 2050 60  0001 C CNN
@@
 $EndComp
 $Comp
-L GND #PWR022
+L GND #PWR17
 U 1 1 53EF7CD3
 P 7800 4450
-F 0 "#PWR022" H 7800 4450 30  0001 C CNN
+F 0 "#PWR17" H 7800 4450 30  0001 C CNN
 F 1 "GND" H 7800 4380 30  0001 C CNN
 F 2 "" H 7800 4450 60  0001 C CNN
@@
 $EndComp
 Wire Wire Line
-	7650 4400 7950 4400
+	7400 4400 7950 4400
 Wire Wire Line
 	7800 4400 7800 4450
 Connection ~ 7800 4400
 Wire Wire Line
-	7650 4000 7950 4000
-$Comp
-L +3.3V #PWR023
+	7400 4000 7950 4000
+$Comp
+L +3.3V #PWR16
 U 1 1 53EF7E3C
 P 7800 3950
-F 0 "#PWR023" H 7800 3910 30  0001 C CNN
+F 0 "#PWR16" H 7800 3910 30  0001 C CNN
 F 1 "+3.3V" H 7800 4060 30  0000 C CNN
 F 2 "" H 7800 3950 60  0001 C CNN
@@
 LCD-contr
 $Comp
-L +3.3V #PWR024
+L +3.3V #PWR15
 U 1 1 53EFB331
 P 6800 3200
-F 0 "#PWR024" H 6800 3160 30  0001 C CNN
+F 0 "#PWR15" H 6800 3160 30  0001 C CNN
 F 1 "+3.3V" H 6800 3310 30  0000 C CNN
 F 2 "" H 6800 3200 60  0001 C CNN
@@
 $EndComp
 $Comp
-L GND #PWR025
+L GND #PWR14
 U 1 1 53F01757
 P 6450 2400
-F 0 "#PWR025" H 6450 2400 30  0001 C CNN
+F 0 "#PWR14" H 6450 2400 30  0001 C CNN
 F 1 "GND" H 6450 2330 30  0001 C CNN
 F 2 "" H 6450 2400 60  0001 C CNN
@@
 	5050 3100 5200 3100
 $Comp
-L +3.3V #PWR026
+L +3.3V #PWR10
 U 1 1 53F0185A
 P 6000 3000
-F 0 "#PWR026" H 6000 2960 30  0001 C CNN
+F 0 "#PWR10" H 6000 2960 30  0001 C CNN
 F 1 "+3.3V" H 6000 3110 30  0000 C CNN
 F 2 "" H 6000 3000 60  0001 C CNN
@@
 	5200 3700 5200 3850
 $Comp
-L +3.3V #PWR027
+L +3.3V #PWR12
 U 1 1 53F040DD
 P 6050 3850
-F 0 "#PWR027" H 6050 3810 30  0001 C CNN
+F 0 "#PWR12" H 6050 3810 30  0001 C CNN
 F 1 "+3.3V" H 6050 3960 30  0000 C CNN
 F 2 "" H 6050 3850 60  0001 C CNN
@@
 	5700 3850 6050 3850
 $Comp
-L GND #PWR028
+L GND #PWR13
 U 1 1 53F04173
 P 6150 3700
-F 0 "#PWR028" H 6150 3700 30  0001 C CNN
+F 0 "#PWR13" H 6150 3700 30  0001 C CNN
 F 1 "GND" H 6150 3630 30  0001 C CNN
 F 2 "" H 6150 3700 60  0001 C CNN
@@
 	9200 3800 9350 3800
 Connection ~ 9200 3700
+$Comp
+L C C9
+U 1 1 53F1220A
+P 7400 4200
+F 0 "C9" H 7400 4300 40  0000 L CNN
+F 1 "C" H 7406 4115 40  0000 L CNN
+F 2 "Capacitors_SMD:c_0805" H 7438 4050 30  0001 C CNN
+F 3 "" H 7400 4200 60  0000 C CNN
+	1    7400 4200
+	1    0    0    -1
+$EndComp
+Connection ~ 7650 4000
+Connection ~ 7650 4400
 $EndSCHEMATC

Commit message: o Get terminal up-to-date with current KiCad libraries o check in cache as it is vital to be backward compatible.
Parts:
- P1: symbol CONN_5 -> CONN_01X05
- P10: symbol CONN_4 -> CONN_01X04
- P11, P14: symbol CONN_5X2 -> CONN_02X05
- P12: symbol CONN_4 -> CONN_02X05
- P13: symbol CONN_3X2 -> CONN_02X03
- P2: symbol CONN_8 -> CONN_01X08
- P3, P4: symbol CONN_8X2 -> CONN_02X08
- P9: symbol CONN_2X2 -> CONN_02X02
Connections:
- wire segments 66 -> 86
Other:
- moved on the sheet: C1, C2, C3, C4, C5, C6, C9, J1
