File: hardware/multi-interface/multi-interface.kicad_pcb (KiCad board)
At the start: 2 copper layers, 70 x 45 mm, 24 parts, among them J1 RJ45, J2 RJ45, J3 RJ45, J4 RJ45, P1 CONN_4X2, P2 CONN_2, P3 CONN_2, P4 CONN_1, P5 CONN_1, P6 CONN_1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

Commit message: o final touches   - ground plane   - reference to Noisebridge and git repository.
Parts:
- moved P6 7.02 mm to (108.0, 108.0)
- moved P7 7.02 mm to (172.0, 108.0)
- moved P4 0.50 mm to (172.0, 90.0)
- moved P5 0.50 mm to (108.0, 90.0)
Routing:
- added copper zone on B.Cu, net GND
- added copper zone on F.Cu, net GND
Other:
- board size 70 x 45 mm -> 70 x 30 mm
- board text added: "CC-BY-SA"
- board text added: "H.Zeller"
- board text added: "Noisebridge"
- board text added: "github.com/hzeller/rfid-access-control"

Commit message: o move mounting hole P6... out of the way. o Add version and 'reboot' designator :)
Other:
- board text added: ""reboot""
- board text added: "v. 0.1"

Commit message: o add year.
Other:
- board text added: "2014"
