File: hardware/multi-interface/multi-interface.sch (KiCad schematic (older format))
At the start: 24 parts, among them J1 RJ45, J2 RJ45, J3 RJ45, J4 RJ45, P1 CONN_4X2, P2 CONN_2, P3 CONN_2, P4 CONN_1, P5 CONN_1, P6 CONN_1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

Commit message: o Re-connect with current KiCad library. o add cache to repository to make sure this is kept.
Parts:
- removed P4, P5, P6, P7: CONN_1, Connect:1pin, symbol CONN_1
- P1: symbol CONN_4X2 -> CONN_02X04
- P2, P3: symbol CONN_2 -> CONN_01X02
Connections:
- wire segments 92 -> 120
Other:
- note removed: "Mounting holes"
- moved on the sheet: C1, C10, C6, C7, C8, C9
